File: ESP32wroom.kicad_pcb (KiCad board)
At the start: 2 copper layers, 32 parts, among them J1 Conn_01x19, J2 USB_C_Receptacle_USB2.0, J3 Conn_01x19, Q1 S8050, Q2 S8050, SW1 SW_SPST, SW2 SW_SPST, U1 ESP32-WROOM-32, U2 AMS1117-3.3, U3 CH340C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

Commit message: Ca
Parts:
- removed D1, D3, D4: SZESD9B5.0ST5G, Diode_SMD:D_SOD-923
- removed D5: ESD5Zxx, Diode_SMD:D_SOD-523
- removed U3: CH340C, Package_SO:SOIC-16_3.9x9.9mm_P1.27mm
- added D6: SS14, Diode_SMD:Nexperia_CFP3_SOD-123W, F.Cu at (132.5, 118.4)
- added R7: 5.1K, Capacitor_SMD:C_0603_1608Metric, F.Cu at (137.1, 113.6)
- added R8: 5.1K, Capacitor_SMD:C_0603_1608Metric, F.Cu at (138.8, 113.6)
- J1, J3: value Conn_01x19 -> Conn_01x16; footprint Connector_PinSocket_2.54mm:PinSocket_1x19_P2.54mm_Vertical -> Connector_PinSocket_2.54mm:PinSocket_1x16_P2.54mm_Vertical
- moved R2 26.8 mm to (151.0, 83.5), turned to 90 degrees
- moved R3 21.6 mm to (151.0, 86.8), turned to 90 degrees
- moved SW1 20.5 mm to (147.5, 123.0)
- moved C6 20.5 mm to (144.9, 122.1)
- moved C5 7.13 mm to (135.0, 106.3), turned to -90 degrees
- moved C4 4.61 mm to (136.6, 103.4)
- moved C7 4.25 mm to (154.1, 122.0)
- moved C3 4.19 mm to (138.1, 103.4)
- moved SW2 4.03 mm to (151.4, 123.0)
- moved R4 3.96 mm to (147.5, 110.7), turned to 180 degrees
- moved R5 3.31 mm to (150.5, 110.5), turned to -90 degrees
- moved Q2 2.74 mm to (147.3, 113.7), turned to 180 degrees
- moved Q1 2.50 mm to (147.2, 107.6), turned to 180 degrees
- moved C10 2.32 mm to (124.5, 80.7)
- moved R6 1.54 mm to (126.0, 80.7)
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Connections:
- J1 pad 1: /VDD3V3 -> +3V3
- J1 pad 14: GND -> /IO13
- J1 pad 15: /IO13 -> GND
- J1 pad 16: /SD2 -> +5V
- J2 pad A5: unconnected-(J2-CC1-PadA5) -> Net-(J2-CC1)
- J2 pad B5: unconnected-(J2-CC2-PadB5) -> Net-(J2-CC2)
- J2 pad S1: unconnected-(J2-SHIELD-PadS1) -> GND
- U1 pad 1: Net-(U1-GND-Pad1) -> GND
- U1 pad 15: Net-(U1-GND-Pad1) -> GND
- U1 pad 38: Net-(U1-GND-Pad1) -> GND
- U1 pad 39: Net-(U1-GND-Pad1) -> GND
- U4 pad 19: /~{RTS} -> /RTS
- U4 pad 23: /~{DTR} -> /DTR
Routing:
- net +3V3: track 0.00 -> 71.2 mm, vias 0 -> 4
- net /EN: track 0.00 -> 63.4 mm, vias 0 -> 2
- net /RXD: track 0.00 -> 36.3 mm, vias 0 -> 2
- net /TXD: track 0.00 -> 34.6 mm
- net /GPIO0: track 0.00 -> 30.9 mm, vias 0 -> 2
- net +5V: track 0.00 -> 29.1 mm
- net /IO15: track 0.00 -> 26.2 mm, vias 0 -> 1
- net /IO2: track 0.00 -> 23.1 mm, vias 0 -> 1
- net /USB_DP: track 0.00 -> 22.2 mm, vias 0 -> 2
- net /USB_DN: track 0.00 -> 21.8 mm, vias 0 -> 2
- net /IO13: track 0.00 -> 21.8 mm
- net /IO4: track 0.00 -> 19.3 mm
- net /IO12: track 0.00 -> 19.2 mm
- net /IO14: track 0.00 -> 18.3 mm
- net /IO16: track 0.00 -> 18.0 mm
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- added copper zone on B.Cu, net GND
- added copper zone on F.Cu, net GND
Other:
- board outline added: 39.4 x 52 mm
- board text added: "BOOT"
- board text added: "IO32"
- board text added: "IO35"
- board text added: "RST"
