File: ESP32wroom.kicad_pcb (KiCad board)
At the start: 2 copper layers, 37.5 x 51.8 mm, 34 parts, among them J1 Conn_01x16, J2 USB_C_Receptacle_USB2.0, J3 Conn_01x16, Q1 S8050, Q2 S8050, SW1 SW_SPST, SW2 SW_SPST, U1 ESP32-WROOM-32, U2 AMS1117-3.3, U4 CH9102F

Commit message: AD
Parts:
- removed C4: 0.1uF, Capacitor_SMD:C_0603_1608Metric
- added G***: LOGO, LOGO, F.Cu at (196.2, 127.6)
- added G***: LOGO, LOGO, F.Cu at (200.7, 127.6)
- added R12: 10K, Resistor_SMD:R_0603_1608Metric, F.Cu at (183.5, 109.6)
- C1, C10, C9: value C -> 0.1uF
- C2, C6, C8: value C -> 10uF
- R10, R11: value R -> 5K
- R4, R5, R6: value R -> 10K
- R9: value R -> 470R
- turned C9 to 0 degrees
Connections:
- C9 pad 1: GND -> +3V3
- C9 pad 2: +3V3 -> GND
- U4 pad 6: Net-(U4-V3) -> +3V3
Routing:
- net +3V3: track 71.4 -> 80.6 mm, vias 5 -> 6
- net Net-(U4-V3): track 2.94 -> 0.00 mm
- net /~{RST}: track 0.00 -> 2.68 mm
- net +5V: track 33.0 -> 35.1 mm, vias 0 -> 2
- net GND: vias 82 -> 79
Other:
- board text removed: "BOOT"
- board text removed: "RST"
