File: ESP32wroom.kicad_sch (KiCad schematic)
At the start: 32 parts, among them J1 Conn_01x19, J2 USB_C_Receptacle_USB2.0, J3 Conn_01x19, Q1 S8050, Q2 S8050, SW1 SW_SPST, SW2 SW_SPST, U1 ESP32-WROOM-32, U2 AMS1117-3.3, U3 CH340C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

Commit message: AD
PCB
Parts:
- C1, C10, C2, C3, C4, C5, C6, C7, C8, C9: footprint (none) -> Capacitor_SMD:C_0603_1608Metric
- D2: footprint (none) -> LED_SMD:LED_0603_1608Metric
- J1, J3: footprint (none) -> Connector_PinSocket_2.54mm:PinSocket_1x19_P2.54mm_Vertical
- J2: footprint (none) -> Connector_USB:USB_C_Receptacle_HRO_TYPE-C-31-M-12
- R1, R2, R3, R5: footprint (none) -> Resistor_SMD:R_0603_1608Metric
Connections:
- net +3.3V is gone; now on net +3V3: C2.1, U2.2 (VO)
- net EXT_5V is gone; now on net +5V: J1.19 (Pin_19)
- net RXD0/IO3 is gone; now on net TXD: U1.34 (RXD0/IO3)
- net TXD0/IO1 is gone; now on net RXD: U1.35 (TXD0/IO1)
- net VDD is gone; now on net +3V3: C3.1, U4.5 (VIO)
- net GPIO0: now also C6.2, SW1.2 (B), U1.25 (IO0)
- net IO0: no longer C6.2, SW1.2 (B), U1.25 (IO0)
Other:
- note added: "Button_Switch_SMD:SW_SPST_B3U-1000P"
- note added: "Capacitor_SMD:C_0603_1608Metric"
- note added: "Connector_PinSocket_2.54mm:PinSocket_1x19_P2.54mm_Vertical"
- note added: "Connector_USB:USB_C_Receptacle_HRO_TYPE-C-31-M-12"
- note added: "Diode_SMD:D_SOD-523"
- note added: "Diode_SMD:D_SOD-923"
- note added: "LED_SMD:LED_0603_1608Metric"
- note added: "Package_TO_SOT_SMD:SC-59"
- note added: "Package_TO_SOT_SMD:SOT-223-3_TabPin2"
- moved on the sheet: C10, R6
Changed lines of the file:
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@@
 	)
 	(junction
-		(at 184.15 39.37)
+		(at 198.12 33.02)
 		(diameter 0)
 		(color 0 0 0 0)
@@
 	(wire
 		(pts
-			(xy 184.15 29.21) (xy 184.15 30.48)
+			(xy 198.12 22.86) (xy 198.12 24.13)
 		)
 		(stroke
@@
 	(wire
 		(pts
-			(xy 184.15 39.37) (xy 191.77 39.37)
+			(xy 198.12 33.02) (xy 205.74 33.02)
 		)
 		(stroke
@@
 	(wire
 		(pts
-			(xy 184.15 48.26) (xy 184.15 46.99)
+			(xy 198.12 41.91) (xy 198.12 40.64)
 		)
 		(stroke
@@
 	(wire
 		(pts
-			(xy 184.15 38.1) (xy 184.15 39.37)
+			(xy 198.12 31.75) (xy 198.12 33.02)
 		)
 		(stroke
@@
 		)
 	)
+	(text "Button_Switch_SMD:SW_SPST_B3U-1000P"
+		(exclude_from_sim no)
+		(at 66.548 124.714 0)
+		(effects
+			(font
+				(size 2.032 2.032)
+			)
+		)
+	)
+	(text "Diode_SMD:D_SOD-923"
+		(exclude_from_sim no)
+		(at 80.01 90.17 0)
+		(effects
+			(font
+				(size 2.032 2.032)
+			)
+		)
+	)
+	(text "Package_TO_SOT_SMD:SC-59"
+		(exclude_from_sim no)
+		(at 43.18 105.664 0)
+		(effects
+			(font
+				(size 2.032 2.032)
+			)
+		)
+	)
+	(text "LED_SMD:LED_0603_1608Metric"
+		(exclude_from_sim no)
+		(at 39.116 48.26 0)
+		(effects
+			(font
+				(size 2.032 2.032)
+			)
+		)
+	)
+	(text "Package_TO_SOT_SMD:SOT-223-3_TabPin2"
+		(exclude_from_sim no)
+		(at 49.53 17.272 0)
+		(effects
+			(font
+				(size 2.032 2.032)
+			)
+		)
+	)
+	(text "Capacitor_SMD:C_0603_1608Metric"
+		(exclude_from_sim no)
+		(at 58.928 37.846 0)
+		(effects
+			(font
+				(size 2.032 2.032)
+			)
+		)
+	)
+	(text "Connector_PinSocket_2.54mm:PinSocket_1x19_P2.54mm_Vertical"
+		(exclude_from_sim no)
+		(at 179.07 102.362 0)
+		(effects
+			(font
+				(size 1.27 1.27)
+			)
+		)
+	)
+	(text "Diode_SMD:D_SOD-523"
+		(exclude_from_sim no)
+		(at 71.374 63.754 0)
+		(effects
+			(font
+				(size 2.032 2.032)
+			)
+		)
+	)
+	(text "Connector_USB:USB_C_Receptacle_HRO_TYPE-C-31-M-12"
+		(exclude_from_sim no)
+		(at 63.5 101.346 0)
+		(effects
+			(font
+				(size 2.032 2.032)
+			)
+		)
+	)
 	(label "IO17"
 		(at 245.11 69.85 0)
@@
 	)
 	(label "EN"
-		(at 189.23 39.37 0)
+		(at 203.2 33.02 0)
 		(fields_autoplaced yes)
 		(effects
@@
 		)
 	)
-	(label "IO0"
+	(label "GPIO0"
 		(at 82.55 137.16 0)
 		(fields_autoplaced yes)
@@
 		)
 	)
-	(label "RXD0/IO3"
+	(label "TXD"
 		(at 245.11 49.53 0)
 		(fields_autoplaced yes)
@@
 		)
 	)
-	(label "IO0"
+	(label "GPIO0"
 		(at 245.11 41.91 0)
 		(fields_autoplaced yes)
@@
 		)
 	)
-	(label "TXD0/IO1"
+	(label "RXD"
 		(at 245.11 44.45 0)
 		(fields_autoplaced yes)
@@
 		)
 	)
-	(label "EXT_5V"
+	(label "+5V"
 		(at 181.61 154.94 180)
 		(fields_autoplaced yes)
@@
 			)
 		)
-		(property "Footprint" ""
+		(property "Footprint" "Connector_PinSocket_2.54mm:PinSocket_1x19_P2.54mm_Vertical"
 			(at 199.39 132.08 0)
 			(effects
@@
 			)
 		)
-		(property "Footprint" ""
+		(property "Footprint" "Connector_PinSocket_2.54mm:PinSocket_1x19_P2.54mm_Vertical"
 			(at 170.18 132.08 0)
 			(effects
@@
 			)
 		)
-		(property "Value" "+3.3V"
-			(at 48.26 22.86 0)
+		(property "Value" "+3V3"
+			(at 48.26 21.59 0)
 			(effects
 				(font
@@
 	(symbol
 		(lib_id "power:+3V3")
-		(at 184.15 29.21 0)
+		(at 198.12 22.86 0)
 		(unit 1)
 		(exclude_from_sim no)
@@
 		(dnp no)
 		(property "Reference" "#PWR020"
-			(at 184.15 33.02 0)
+			(at 198.12 26.67 0)
 			(effects
 				(font
@@
 		)
 		(property "Value" "+3V3"
-			(at 186.69 28.194 0)
+			(at 200.66 21.844 0)
 			(effects
 				(font
@@
 		)
 		(property "Footprint" ""
-			(at 184.15 29.21 0)
+			(at 198.12 22.86 0)
 			(effects
 				(font
@@
 		)
 		(property "Datasheet" ""
-			(at 184.15 29.21 0)
+			(at 198.12 22.86 0)
 			(effects
 				(font
@@
 		)
 		(property "Description" ""
-			(at 184.15 29.21 0)
+			(at 198.12 22.86 0)
 			(effects
 				(font
@@
 	(symbol
 		(lib_id "Device:R")
-		(at 184.15 34.29 180)
+		(at 198.12 27.94 180)
 		(unit 1)
 		(exclude_from_sim no)
@@
 		(fields_autoplaced yes)
 		(property "Reference" "R6"
-			(at 186.69 33.0199 0)
+			(at 200.66 26.6699 0)
 			(effects
 				(font
@@
 		)
 		(property "Value" "R"
-			(at 186.69 35.5599 0)
+			(at 200.66 29.2099 0)
 			(effects
 				(font
@@
 		)
 		(property "Footprint" "Resistor_SMD:R_0603_1608Metric"
-			(at 185.928 34.29 90)
+			(at 199.898 27.94 90)
 			(effects
 				(font
@@
 		)
 		(property "Datasheet" "~"
-			(at 184.15 34.29 0)
+			(at 198.12 27.94 0)
 			(effects
 				(font
@@
 		)
 		(property "Description" ""
-			(at 184.15 34.29 0)
+			(at 198.12 27.94 0)
 			(effects
 				(font
@@
 			)
 		)
-		(property "Footprint" ""
+		(property "Footprint" "Capacitor_SMD:C_0603_1608Metric"
 			(at 80.01 152.7048 0)
 			(effects
@@
 	(symbol
 		(lib_id "power:GND")
-		(at 184.15 48.26 0)
+		(at 198.12 41.91 0)
 		(unit 1)
 		(exclude_from_sim no)
@@
 		(dnp no)
 		(property "Reference" "#PWR019"
-			(at 184.15 54.61 0)
+			(at 198.12 48.26 0)
 			(effects
 				(font
@@
 		)
 		(property "Value" "GND"
-			(at 184.15 52.324 0)
+			(at 198.12 45.974 0)
 			(effects
 				(font
@@
 		)
 		(property "Footprint" ""
-			(at 184.15 48.26 0)
+			(at 198.12 41.91 0)
 			(effects
 				(font
@@
 		)
 		(property "Datasheet" ""
-			(at 184.15 48.26 0)
+			(at 198.12 41.91 0)
 			(effects
 				(font
@@
 		)
 		(property "Description" ""
-			(at 184.15 48.26 0)
+			(at 198.12 41.91 0)
 			(effects
 				(font
@@
 			)
 		)
-		(property "Footprint" ""
+		(property "Footprint" "Resistor_SMD:R_0603_1608Metric"
 			(at 43.18 156.718 90)
 			(effects
@@
 			)
 		)
-		(property "Footprint" ""
+		(property "Footprint" "Capacitor_SMD:C_0603_1608Metric"
 			(at 49.2252 34.29 0)
 			(effects
@@
 			)
 		)
-		(property "Footprint" ""
+		(property "Footprint" "Capacitor_SMD:C_0603_1608Metric"
 			(at 129.54 20.6248 0)
 			(effects
@@
 			)
 		)
-		(property "Footprint" ""
+		(property "Footprint" "Capacitor_SMD:C_0603_1608Metric"
 			(at 128.27 25.7048 0)
 			(effects
@@
 			)
 		)
-		(property "Footprint" ""
+		(property "Footprint" "Resistor_SMD:R_0603_1608Metric"
 			(at 18.542 30.48 90)
 			(effects
@@
 			)
 		)
-		(property "Value" "VDD"
+		(property "Value" "+3V3"
 			(at 121.666 16.764 0)
 			(effects
@@
 			)
 		)
-		(property "Footprint" ""
+		(property "Footprint" "Capacitor_SMD:C_0603_1608Metric"
 			(at 224.79 26.9748 0)
 			(effects
@@
 			)
 		)
-		(property "Footprint" ""
+		(property "Footprint" "Resistor_SMD:R_0603_1608Metric"
 			(at 43.18 149.098 90)
 			(effects
@@
 			)
 		)
-		(property "Footprint" ""
+		(property "Footprint" "Capacitor_SMD:C_0603_1608Metric"
 			(at 224.79 32.0548 0)
 			(effects
@@
 			)
 		)
-		(property "Footprint" ""
+		(property "Footprint" "Connector_USB:USB_C_Receptacle_HRO_TYPE-C-31-M-12"
 			(at 31.75 73.66 0)
 			(effects
@@
 			)
 		)
-		(property "Footprint" ""
+		(property "Footprint" "Resistor_SMD:R_0603_1608Metric"
 			(at 45.72 131.318 90)
 			(effects
@@
 			)
 		)
-		(property "Footprint" ""
+		(property "Footprint" "Capacitor_SMD:C_0603_1608Metric"
 			(at 80.01 141.2748 0)
 			(effects
@@
 			)
 		)
-		(property "Footprint" ""
+		(property "Footprint" "LED_SMD:LED_0603_1608Metric"
 			(at 20.32 38.1 0)
 			(effects
@@
 			)
 		)
-		(property "Footprint" ""
+		(property "Footprint" "Capacitor_SMD:C_0603_1608Metric"
 			(at 106.68 35.8648 0)
 			(effects
@@
 			)
 		)
-		(property "Footprint" ""
+		(property "Footprint" "Capacitor_SMD:C_0603_1608Metric"
 			(at 27.6352 35.56 0)
 			(effects
@@
 	(symbol
 		(lib_id "Device:C")
-		(at 184.15 43.18 0)
+		(at 198.12 36.83 0)
 		(unit 1)
 		(exclude_from_sim no)
@@
 		(fields_autoplaced yes)
 		(property "Reference" "C10"
-			(at 187.96 41.9099 0)
+			(at 201.93 35.5599 0)
 			(effects
 				(font
@@
 		)
 		(property "Value" "C"
-			(at 187.96 44.4499 0)
+			(at 201.93 38.0999 0)
 			(effects
 				(font
@@
 			)
 		)
-		(property "Footprint" ""
-			(at 185.1152 46.99 0)
+		(property "Footprint" "Capacitor_SMD:C_0603_1608Metric"
+			(at 199.0852 40.64 0)
 			(effects
 				(font
@@
 		)
 		(property "Datasheet" "~"
-			(at 184.15 43.18 0)
+			(at 198.12 36.83 0)
 			(effects
 				(font
@@
 		)
 		(property "Description" ""
-			(at 184.15 43.18 0)
+			(at 198.12 36.83 0)
 			(effects
 				(font

Commit message: Ca
Parts:
- removed D1, D3, D4: SZESD9B5.0ST5G, Diode_SMD:D_SOD-923, symbol Diode:SZESD9B5.0ST5G
- removed D5: ESD5Zxx, Diode_SMD:D_SOD-523, symbol Diode:ESD5Zxx
- removed J1, J3: Conn_01x19, Connector_PinSocket_2.54mm:PinSocket_1x19_P2.54mm_Vertical, symbol Connector_Generic:Conn_01x19
- added D6: SS14, Diode_SMD:Nexperia_CFP3_SOD-123W, symbol Diode:SS14
- added J1, J3: Conn_01x16, Connector_PinSocket_2.54mm:PinSocket_1x16_P2.54mm_Vertical, symbol Connector_Generic:Conn_01x16
- added R7, R8: 5.1K, Capacitor_SMD:C_0603_1608Metric, symbol Device:R
Connections:
- net ~{DTR} is gone; now on net DTR: U4.23 (~{DTR})
- net ~{RTS} is gone; now on net RTS: U4.19 (~{RTS})
- net +3V3: now also J1.1 (Pin_1)
- net +5V: now also D6.1 (K), J1.16 (Pin_16)
- net EN: now also J1.2 (Pin_2)
- net GND: now also J2.S1 (SHIELD), U1.1 (GND), U1.15 (GND), U1.38 (GND), U1.39 (GND), J1.15 (Pin_15), J3.1 (Pin_1), J3.7 (Pin_7), R7.2, R8.2
- net IO0: now also J3.14 (Pin_14)
- net IO12: now also J1.13 (Pin_13)
- net IO13: now also J1.14 (Pin_14)
- net IO14: now also J1.12 (Pin_12)
- net IO15: now also J3.16 (Pin_16)
- net IO16: now also J3.12 (Pin_12)
- net IO17: now also J3.11 (Pin_11)
- net IO18: now also J3.9 (Pin_9)
- net IO19: now also J3.8 (Pin_8)
- net IO2: now also J3.15 (Pin_15)
- net IO21: now also J3.6 (Pin_6)
- net IO22: now also J3.3 (Pin_3)
- net IO23: now also J3.2 (Pin_2)
- net IO25: now also J1.9 (Pin_9)
- net IO26: now also J1.10 (Pin_10)
- net IO27: now also J1.11 (Pin_11)
- net IO32: now also J1.7 (Pin_7)
- net IO33: now also J1.8 (Pin_8)
- net IO34: now also J1.5 (Pin_5)
- net IO35: now also J1.6 (Pin_6)
- net IO4: now also J3.13 (Pin_13)
- net IO5: now also J3.10 (Pin_10)
- net RXD0: now also J3.5 (Pin_5)
- net SENSOR_VN: now also J1.4 (Pin_4)
- net SENSOR_VP: now also J1.3 (Pin_3)
- net TXD0: now also J3.4 (Pin_4)
- net at J2.A4 (VBUS), J2.A9 (VBUS), J2.B4 (VBUS)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: now also D6.2 (A)
- net at J2.A5 (CC1): now also R7.1
- net at J2.B5 (CC2): now also R8.1
Other:
- note added: "Diode_SMD:Nexperia_CFP3_SOD-123W"
- note removed: "Diode_SMD:D_SOD-923"
