File: ESP32wroom.kicad_sch (KiCad schematic)
At the start: 32 parts, among them J1 Conn_01x19, J2 USB_C_Receptacle_USB2.0, J3 Conn_01x19, Q1 S8050, Q2 S8050, SW1 SW_SPST, SW2 SW_SPST, U1 ESP32-WROOM-32, U2 AMS1117-3.3, U3 CH340C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

Commit message: AD
Parts:
- removed C9: C, symbol Device:C
- removed D1, D3, D4: SZESD9B5.0ST5G, Diode_SMD:D_SOD-923, symbol Diode:SZESD9B5.0ST5G
- removed D5: ESD5Zxx, Diode_SMD:D_SOD-523, symbol Diode:ESD5Zxx
- removed J1, J3: Conn_01x19, symbol Connector_Generic:Conn_01x19
- removed R2, R3: 0R, symbol Device:R
- added D1: LED, LED_SMD:LED_0603_1608Metric, symbol Device:LED
- added D6: SS14, Diode_SMD:Nexperia_CFP3_SOD-123W, symbol Diode:SS14
- added J1, J3: Conn_01x16, Connector_PinSocket_2.54mm:PinSocket_1x16_P2.54mm_Vertical, symbol Connector_Generic:Conn_01x16
- added R10, R11, R9: R, Resistor_SMD:R_0603_1608Metric, symbol Device:R
- added R7, R8: 5.1K, Capacitor_SMD:C_0603_1608Metric, symbol Device:R
- C1, C10, C2, C3, C4, C5, C7, C8: footprint (none) -> Capacitor_SMD:C_0603_1608Metric
- C6: value 0.1uF -> C; footprint (none) -> Capacitor_SMD:C_0603_1608Metric
- D2: footprint (none) -> LED_SMD:LED_0603_1608Metric
- J2: footprint (none) -> Connector_USB:USB_C_Receptacle_HRO_TYPE-C-31-M-12
- R1, R5: footprint (none) -> Resistor_SMD:R_0603_1608Metric
Connections:
- net +3.3V is gone; now on net +3V3: C2.1, U2.2 (VO)
- net GPIO0 is gone; now on net IO0: Q1.3 (C)
- net RXD0/IO3 is gone; now on net TXD: U1.34 (RXD0/IO3)
- net TXD0/IO1 is gone; now on net RXD: U1.35 (TXD0/IO1)
- net VDD is gone; now on net +3V3: C3.1, U4.5 (VIO)
- net ~{DTR} is gone; now on net DTR: U4.23 (~{DTR})
- net ~{RTS} is gone; now on net RTS: U4.19 (~{RTS})
- net +3V3: now also J1.1 (Pin_1), R10.1, R9.1; no longer C8.2
- net +5V: now also C6.2, C8.2, D6.1 (K), J1.16 (Pin_16)
- net EN: now also J1.2 (Pin_2)
- net GND: now also J2.S1 (SHIELD), U1.1 (GND), U1.15 (GND), U1.38 (GND), U1.39 (GND), J1.15 (Pin_15), J3.1 (Pin_1), J3.16 (Pin_16), R11.2, R7.2, R8.2
- net IO0: now also J3.13 (Pin_13), R10.2; no longer C6.2
- net IO12: now also J1.13 (Pin_13)
- net IO13: now also D1.1 (K), J1.14 (Pin_14)
- net IO14: now also J1.12 (Pin_12)
- net IO15: now also J3.15 (Pin_15)
- net IO16: now also J3.11 (Pin_11)
- net IO17: now also J3.10 (Pin_10)
- net IO18: now also J3.8 (Pin_8)
- net IO19: now also J3.7 (Pin_7)
- net IO2: now also J3.14 (Pin_14), R11.1
- net IO21: now also J3.6 (Pin_6)
- net IO22: now also J3.3 (Pin_3)
- net IO23: now also J3.2 (Pin_2)
- net IO25: now also J1.9 (Pin_9)
- net IO26: now also J1.10 (Pin_10)
- net IO27: now also J1.11 (Pin_11)
- net IO32: now also J1.7 (Pin_7)
- net IO33: now also J1.8 (Pin_8)
- net IO34: now also J1.5 (Pin_5)
- net IO35: now also J1.6 (Pin_6)
- net IO4: now also J3.12 (Pin_12)
- net IO5: now also J3.9 (Pin_9)
- net RXD: now also J3.4 (Pin_4)
- net SENSOR_VN: now also J1.4 (Pin_4)
- net SENSOR_VP: now also J1.3 (Pin_3)
- net TXD: now also J3.5 (Pin_5)
- net at J2.A4 (VBUS), J2.A9 (VBUS), J2.B4 (VBUS)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: now also D6.2 (A)
- net at J2.A5 (CC1): now also R7.1
- net at J2.B5 (CC2): now also R8.1
- new net: D1.2 (A), R9.2
Other:
- note added: "Button_Switch_SMD:SW_SPST_B3U-1000P"
- note added: "Capacitor_SMD:C_0603_1608Metric"
- note added: "Connector_PinSocket_2.54mm:PinSocket_1x19_P2.54mm_Vertical"
- note added: "Connector_USB:USB_C_Receptacle_HRO_TYPE-C-31-M-12"
- note added: "Diode_SMD:D_SOD-523"
- note added: "Diode_SMD:Nexperia_CFP3_SOD-123W"
- note added: "LED_SMD:LED_0603_1608Metric"
- note added: "Package_TO_SOT_SMD:SC-59"
- note added: "Package_TO_SOT_SMD:SOT-223-3_TabPin2"
- moved on the sheet: C10, D2, R1, R6, SW1
