File: ESP32wroom.kicad_sch (KiCad schematic)
At the start: 32 parts, among them J1 Conn_01x16, J2 USB_C_Receptacle_USB2.0, J3 Conn_01x16, Q1 S8050, Q2 S8050, SW1 SW_SPST, SW2 SW_SPST, U1 ESP32-WROOM-32, U2 AMS1117-3.3, U3 CH340C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

Commit message: AD
Parts:
- removed C4: 0.1uF, Capacitor_SMD:C_0603_1608Metric, symbol Device:C
- added C9: 0.1uF, Capacitor_SMD:C_0603_1608Metric, symbol Device:C
- added R12: 10K(NC), Resistor_SMD:R_0603_1608Metric, symbol Device:R
- C1, C10: value C -> 0.1uF
- C2, C6, C8: value C -> 10uF
- R10, R11: value R -> 5K
- R4, R5, R6: value R -> 10K
- R9: value R -> 470R
Connections:
- net +3V3: now also U4.6 (V3), C9.1, R12.2
- net GND: now also C9.2
- net ~{RST}: now also R12.1
Other:
- moved on the sheet: C3, Q1, Q2, R4, R5
